Commit message: add ls lidar params and change eular to quaternion

File: launch/include/config/scout.urdf.xacro (robot description, xacro)
@@ -4,13 +4,13 @@
   <link name="base_link"></link>
   <link name="base_imu"> </link>
-  <joint name="imu_joint" type="fixed">
+  <joint name="base_imu_joint" type="fixed">
     <parent link="base_link" />
     <child link="base_imu" />
-    <origin xyz="0 0 0.0405" rpy="0 0 0" />
+    <origin xyz="0.011 0 0" rpy="0 0 0" />
   </joint>
-  <link name="base_scan_3d"> </link>
-  <joint name="velodyne_joint" type="fixed">
+  <link name="base_lidar"> </link>
+  <joint name="base_lidar_joint" type="fixed">
     <parent link="base_link" />
-    <child link="base_scan_3d" />
+    <child link="base_lidar" />
     <origin xyz="0 0 0" rpy="0 0 0" />
   </joint>

Commit message: add kSCFilterSize

File: launch/include/config/scout.urdf.xacro (robot description, xacro)
@@ -15,3 +15,9 @@
     <origin xyz="0 0 0" rpy="0 0 0" />
   </joint>
+  <link name="base_gnss"> </link>
+  <joint name="base_gnss_joint" type="fixed">
+    <parent link="base_link" />
+    <child link="base_gnss" />
+    <origin xyz="-0.30286 0.0 0.614498" rpy="0 0 0"/>
+  </joint>
 </robot>
